File: Hardware-designs/Gateway_v1.1/Gateway_v1.1.kicad_sch (KiCad schematic)
At the start: 39 parts, among them J1 UART, J3 USB_C, J4 UART, SW1 main, SW2 Aux, U1 ESP32-TCP, U2 AMS1117, U3 AMS1117, U4 ESP32-NOW

Commit message: Add pcb images, step file, and pdf schematic for all hardware designs.
Parts:
- removed R14: 330, Resistor_SMD:R_1206_3216Metric_Pad1.30x1.75mm_HandSolder, symbol Device:R
- removed R15: 1.8k, Resistor_SMD:R_1206_3216Metric_Pad1.30x1.75mm_HandSolder, symbol Device:R
- removed R16: 1k, Resistor_SMD:R_1206_3216Metric_Pad1.30x1.75mm_HandSolder, symbol Device:R
- removed R3: 10k, Resistor_SMD:R_1206_3216Metric_Pad1.30x1.75mm_HandSolder, symbol Device:R
Connections:
- net at J4.2 (Pin_2): now also U4.35 (TXD0/IO1)
- net at U4.34 (RXD0/IO3): now also J4.3 (Pin_3)
Other:
- title: (none) -> HueMix-Link Gateway

Commit message: Minor KiCad files update for all devices
Parts:
- C3, C9: value 1nF -> 68nF
Changed lines of the file:
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@@
 			)
 		)
-		(property "Value" "1nF"
+		(property "Value" "68nF"
 			(at 36.83 38.0999 0)
 			(effects
@@
 			)
 		)
-		(property "Value" "1nF"
+		(property "Value" "68nF"
 			(at 33.02 170.1799 0)
 			(effects
