File: Hardware-designs/Lightstrip_m5_v1/Lightstrip_m5_v1.kicad_pcb (KiCad board)
At the start: 2 copper layers, 55 x 36 mm, 22 parts, among them J1 In 24V, J2 lamps, J3 UART, Q1 AO3400A, SW1 PTS526 SM15 SMTR2 LFS, SW2 PTS526 SM15 SMTR2 LFS, U1 TPS560430X3FDBVT, U2 ESP32-WROOM-32E

Commit message: Add serial labels on pcb
Parts:
- R1: value 200k -> 10K
Other:
- board text added: "3.3V"
- board text added: "GND"
- board text added: "RX"
- board text added: "TX"
Changed lines of the file:
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@@
 			)
 		)
-		(property "Value" "200k"
+		(property "Value" "10K"
 			(at 0 1.83 90)
 			(layer "F.Fab")
@@
 		(layer "Edge.Cuts")
 	)
+	(gr_text "GND"
+		(at 223.85 77.375 0)
+		(layer "F.SilkS")
+		(effects
+			(font
+				(size 0.8 0.8)
+				(thickness 0.1)
+			)
+			(justify left bottom)
+		)
+	)
 	(gr_text "GND PWM RGB 24V"
 		(at 185.51 98.13 90)
@@
 		)
 	)
+	(gr_text "TX"
+		(at 221.625 77.375 0)
+		(layer "F.SilkS")
+		(effects
+			(font
+				(size 0.8 0.8)
+				(thickness 0.1)
+			)
+			(justify left bottom)
+		)
+	)
+	(gr_text "3.3V\n"
+		(at 216.3 77.375 0)
+		(layer "F.SilkS")
+		(effects
+			(font
+				(size 0.8 0.8)
+				(thickness 0.1)
+			)
+			(justify left bottom)
+		)
+	)
 	(gr_text "+"
 		(at 225.69 90.16 0)
@@
 			)
 			(justify left bottom)
+		)
+	)
+	(gr_text "RX"
+		(at 219.45 77.375 0)
+		(layer "F.SilkS")
+		(effects
+			(font
+				(size 0.8 0.8)
+				(thickness 0.1)
+			)
+			(justify left bottom)

Commit message: Minor KiCad files update for all devices
Parts:
- C1: value 100nF -> 68nF
Changed lines of the file:
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@@
 		(embedded_fonts no)
 		(model "${KICAD9_3DMODEL_DIR}/TerminalBlock_Phoenix.3dshapes/TerminalBlock_Phoenix_MKDS-1,5-4_1x04_P5.00mm_Horizontal.step"
+			(hide yes)
 			(offset
 				(xyz 15 0 0)
@@
 			)
 		)
-		(property "Value" "100nF"
+		(property "Value" "68nF"
 			(at 0 1.43 90)
 			(layer "F.Fab")
@@
 		(embedded_fonts no)
 		(model "${KICAD9_3DMODEL_DIR}/TerminalBlock_Phoenix.3dshapes/TerminalBlock_Phoenix_MKDS-1,5-2_1x02_P5.00mm_Horizontal.step"
+			(hide yes)
 			(offset
 				(xyz 0 0 0)
