File: Hardware-designs/Lightstrip_m5_v1/Lightstrip_m5_v1.kicad_sch (KiCad schematic)
At the start: 22 parts, among them J1 In 24V, J2 lamps, J3 UART, Q1 AO3400A, SW1 PTS526 SM15 SMTR2 LFS, SW2 PTS526 SM15 SMTR2 LFS, U1 TPS560430X3FDBVT, U2 ESP32-WROOM-32E

Commit message: Add pcb images, step file, and pdf schematic for all hardware designs.
Other:
- title: (none) -> HueMix-Link Lightstrip Model 5
Changed lines of the file:
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@@
 	(generator_version "9.0")
 	(paper "A4")
+	(title_block
+		(title "HueMix-Link Lightstrip Model 5")
+		(date "2026-02-18")
+		(rev "1.0")
+	)
 	(junction
 		(at 224.79 86.36)

Commit message: add motion sensor hardware
Parts:
- R1: value 200k -> 10K
Changed lines of the file:
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@@
 			)
 		)
-		(property "Value" "200k"
+		(property "Value" "10K"
 			(at 152.4 35.56 90)
 			(effects

Commit message: Minor KiCad files update for all devices
Parts:
- C1: value 100nF -> 68nF
Changed lines of the file:
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@@
 			)
 		)
-		(property "Value" "100nF"
+		(property "Value" "68nF"
 			(at 149.86 44.4499 90)
 			(effects
