File: Hardware-designs/Motion_Sensor_v1.1/Motion_Sensor_v1.1.kicad_sch (KiCad schematic)
At the start: 37 parts, among them J1 UART, J2 Bat, J3 USB_C, J4 I2C, J5 I2C, Q1 AO3407A, SW2 PTS526 SM15 SMTR2 LFS, U1 ESP32-WROOM-32, U2 TP4057, U4 MCP1700

Commit message: correction voltage regulator
Parts:
- U4: footprint MCP1700T_3302E_TT 3:SOT-23_MC_MCH -> PCM_Package_TO_SOT_SMD_AKL:SOT-23; symbol Regulator_Linear:MCP1700-3302E_TO92 -> PCM_Voltage_Regulator_AKL:MCP1700T-3302E-TT
Other:
- moved on the sheet: U4
Changed lines of the file:
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@@
 	(wire
 		(pts
-			(xy 195.58 31.75) (xy 195.58 36.83)
+			(xy 195.58 30.48) (xy 195.58 36.83)
 		)
 		(stroke
@@
 	)
 	(symbol
-		(lib_id "Regulator_Linear:MCP1700-3302E_TO92")
-		(at 195.58 24.13 180)
+		(lib_id "PCM_Voltage_Regulator_AKL:MCP1700T-3302E-TT")
+		(at 195.58 24.13 0)
 		(unit 1)
 		(exclude_from_sim no)
@@
 			)
 		)
-		(property "Footprint" "MCP1700T_3302E_TT 3:SOT-23_MC_MCH"
-			(at 195.58 19.05 0)
-			(effects
-				(font
-					(size 1.27 1.27)
-					(italic yes)
-				)
-				(hide yes)
-			)
-		)
-		(property "Datasheet" "http://ww1.microchip.com/downloads/en/DeviceDoc/20001826D.pdf"
+		(property "Footprint" "PCM_Package_TO_SOT_SMD_AKL:SOT-23"
 			(at 195.58 24.13 0)
 			(effects
@@
 			)
 		)
-		(property "Description" ""
+		(property "Datasheet" "https://ww1.microchip.com/downloads/en/DeviceDoc/MCP1700-Low-Quiescent-Current-LDO-20001826E.pdf"
 			(at 195.58 24.13 0)
 			(effects
@@
 					(size 1.27 1.27)
 				)
-			)
-		)
+				(hide yes)
+			)
+		)
+		(property "Description" "SOT-23 3.3V 250mA Low dropout 3-terminal voltage regulator, Alternate KiCad Library"
+			(at 195.58 24.13 0)
+			(effects
+				(font
+					(size 1.27 1.27)
+				)
+				(hide yes)
+			)
+		)

Commit message: Magnetic Sensor
Parts:
- R14: value 300 -> 300k
Changed lines of the file:
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@@
 			)
 		)
-		(property "Value" "300"
+		(property "Value" "300k"
 			(at 254 125.73 0)
 			(effects

Commit message: Minor KiCad files update for all devices
Parts:
- C3: value 1nF -> 68nF
- R7: value 68k -> 75k
Changed lines of the file:
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@@
 			)
 		)
-		(property "Value" "1nF"
+		(property "Value" "68nF"
 			(at 25.4 40.6399 0)
 			(effects
@@
 			)
 		)
-		(property "Value" "68k"
+		(property "Value" "75k"
 			(at 195.58 142.2399 0)
 			(effects
