File: Hardware-designs/Motion_Sensor_v1.1/Motion_Sensor_v1.1.kicad_pcb (KiCad board)
At the start: 2 copper layers, 57 x 57 mm, 37 parts, among them J1 UART, J2 Bat, J3 USB_C, J4 I2C, J5 I2C, Q1 AO3407A, SW2 PTS526 SM15 SMTR2 LFS, U1 ESP32-WROOM-32, U2 TP4057, U4 MCP1700

Commit message: Magnetic Sensor AAA battery version added
Parts:
- added C7: 100nF, Capacitor_SMD:C_0805_2012Metric_Pad1.18x1.45mm_HandSolder, B.Cu at (66.5, 87.0)
Routing:
- net GND: track 232.2 -> 236.3 mm
- net +3.3V: track 125.0 -> 127.4 mm
