File: Hardware-designs/Lightstrip/Lightstrip.kicad_pcb (KiCad board)
At the start: 2 copper layers, 55 x 36 mm, 22 parts, among them J1 In 24V, J2 lamps, J3 UART, Q1 AO3400A, SW1 PTS526 SM15 SMTR2 LFS, SW2 PTS526 SM15 SMTR2 LFS, U1 TPS560430X3FDBVT, U2 ESP32-WROOM-32E

Commit message: Lightstrip version 2
Parts:
- removed J2: lamps, TerminalBlock:TerminalBlock_MaiXu_MX126-5.0-04P_1x04_P5.00mm
- added J4: lamps, TerminalBlock:TerminalBlock_MaiXu_MX126-5.0-05P_1x05_P5.00mm, F.Cu at (187.1, 77.7)
- added Q2: AO3400A, AO3400A:SOT95P280X125-3N, F.Cu at (194.2, 96.3)
- added R5: 100, Resistor_SMD:R_1206_3216Metric_Pad1.30x1.75mm_HandSolder, F.Cu at (198.2, 96.1)
- moved Q1 5.36 mm to (202.1, 96.2)
- moved R2 5.07 mm to (205.8, 95.9)
- moved C1 4.65 mm to (193.1, 77.4)
- moved R1 2.20 mm to (188.4, 73.0), turned to 180 degrees
Connections:
- net Net-(U2-IO27) renamed Button
- R2 pad 1: Net-(U2-IO26) -> Net-(U2-IO25)
- U2 pad 10: unconnected-(U2-IO25-Pad10) -> Net-(U2-IO25)
Routing:
- net GND: track 204.0 -> 173.9 mm, vias 87 -> 115
- net Net-(U2-IO25): track 0.00 -> 24.1 mm
- net Net-(J4-Pin_3): track 10.6 -> 20.9 mm
- net Net-(J4-Pin_4): track 0.00 -> 8.06 mm
- net Net-(J4-Pin_2): track 49.7 -> 56.7 mm
- net Net-(U2-EN): track 20.0 -> 13.3 mm
- net +24V: track 75.2 -> 81.5 mm
- net Net-(Q2-Pad1): track 0.00 -> 6.15 mm
- net +3.3V: track 83.4 -> 80.6 mm
- net Net-(Q1-Pad1): track 5.94 -> 6.47 mm
Other:
- board text added: "GND PWM1 PWM2 RGB 24V"
- board text added: "LightStrip Version 2 April 2026 HueMix Link"
- board text removed: "GND PWM RGB 24V"
- board text removed: "LightStrip model 5 Version 1 February 2026 HueMix Link"
