File: Hardware-designs/Magnetic Sensor/Magnetic Sensor.kicad_pcb (KiCad board)
At the start: 2 copper layers, 25 x 80 mm, 35 parts, among them J1 UART, J2 JST_02, J3 JST_05, Q1 AO3407A, SW1 SW_Reed_Opener, SW2 PTS526 SM15 SMTR2 LFS, U1 ESP32-WROOM-32, U2 TPS63021DSJR

Commit message: Magnetic sensor update
Parts:
- R1: value 10k -> 270k
Connections:
- U2 pad 13: Net-(U2-EN) -> GND
Routing:
- net GND: track 142.6 -> 143.5 mm
- net Net-(U2-EN): track 12.0 -> 11.5 mm
Other:
- board text added: "HueMix Link Magnetic Sensor v1.01 March 2026"
Changed lines of the file:
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@@
 		)
 		(embedded_fonts no)
-		(model "/Users/gmixich/OneDrive/github/HueMix-Link-V3/Hardware-designs/Magnetic Sensor/components/C1608X5R1A226M080AC/C1608X5R1A226M080AC.step"
+		(model "${KIPRJMOD}/components/C1608X5R1A226M080AC/C1608X5R1A226M080AC.step"
 			(offset
 				(xyz 0 -0.5 0)
@@
 			(size 0.6 0.24)
 			(layers "F.Cu" "F.Paste")
-			(net 5 "Net-(U2-EN)")
+			(net 1 "GND")
 			(pinfunction "PS/SYNC")
 			(pintype "input")
@@
 		)
 		(embedded_fonts no)
-		(model "/Users/gmixich/OneDrive/github/HueMix-Link-V3/Hardware-designs/Magnetic Sensor/components/TPS63021DSJR/TPS63021DSJR.step"
+		(model "${KIPRJMOD}/components/TPS63021DSJR/TPS63021DSJR.step"
 			(offset
 				(xyz 0 0 0)
@@
 		(tags "resistor handsolder")
 		(property "Reference" "R7"
-			(at 0.025 0 -90)
+			(at 0.025 0 270)
 			(layer "B.SilkS")
 			(effects
@@
 			)
 		)
-		(property "Value" "10k"
+		(property "Value" "270k"
 			(at 0 1.65 0)
 			(layer "F.Fab")
@@
 		)
 		(property "Datasheet" "~"
-			(at 0 0 -90)
+			(at 0 0 270)
 			(unlocked yes)
 			(layer "B.Fab")
@@
 		)
 		(property "Description" "3-pole Solder Jumper, pins 1+2 closed/bridged"
-			(at 0 0 -90)
+			(at 0 0 270)
 			(unlocked yes)
 			(layer "B.Fab")
@@
 		(at 117.875 92.275 90)
 		(property "Reference" "BT1"
-			(at -20.775 13.275 -90)
+			(at -20.775 13.275 270)
 			(layer "B.SilkS")
 			(effects
@@
 		)
 		(embedded_fonts no)
-		(model "/Users/gmixich/OneDrive/github/HueMix-Link-V3/Hardware-designs/Magnetic Sensor/components/BH123A/BH123A.step"
+		(model "${KIPRJMOD}/components/BH123A/BH123A.step"
 			(offset
 				(xyz 0 0 0)
@@
 		)
 		(embedded_fonts no)
-		(model "/Users/gmixich/OneDrive/github/HueMix-Link-V3/Hardware-designs/Magnetic Sensor/components/PTS526_SM15_SMTR2_LFS/PTS526SK15SMTR2_LFS.stp"
+		(model "${KIPRJMOD}/components/PTS526_SM15_SMTR2_LFS/PTS526SK15SMTR2_LFS.stp"
 			(offset
 				(xyz 0 0 0)
@@
 		)
 	)
+	(gr_text "HueMix Link\nMagnetic Sensor v1.01\nMarch 2026\n"
+		(at 123.15 98.875 90)
+		(layer "F.SilkS")
+		(effects
+			(font
+				(size 1.25 1.25)
+				(thickness 0.2)
+			)
+			(justify bottom)
+		)
+	)
 	(gr_text "RX"
 		(at 128.65 80.16 90)
@@
 	)
 	(segment
+		(start 121.325 78.3)
+		(end 120.425 78.3)
+		(width 0.2)
+		(layer "F.Cu")
+		(net 1)
+	)
+	(segment
 		(start 123.775 81.734298)
 		(end 123.775 80.9875)
@@
 		(layer "F.Cu")
 		(net 5)
-	)
-	(segment
-		(start 121.325 78.8)
-		(end 121.325 78.3)
-		(width 0.25)
-		(layer "F.Cu")
-		(net 5)

Commit message: Minor KiCad files update for all devices
Parts:
- C3: value 1nF -> 68nF
- R1: value 270k -> 200k
- R7: value 68k -> 75k
Changed lines of the file:
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@@
 			)
 		)
-		(property "Value" "1nF"
+		(property "Value" "68nF"
 			(at 0 1.68 90)
 			(layer "F.Fab")
@@
 			)
 		)
-		(property "Value" "68k"
+		(property "Value" "75k"
 			(at 0 1.65 90)
 			(layer "F.Fab")
@@
 			)
 		)
-		(property "Value" "270k"
+		(property "Value" "200k"
 			(at 0 1.65 0)
 			(layer "F.Fab")
