File: Hardware-designs/Magnetic Sensor/Magnetic Sensor.kicad_sch (KiCad schematic)
At the start: 35 parts, among them J1 UART, J2 JST_02, J3 JST_05, Q1 AO3407A, SW1 SW_Reed_Opener, SW2 PTS526 SM15 SMTR2 LFS, U1 ESP32-WROOM-32, U2 TPS63021DSJR

Commit message: Magnetic sensor update
Parts:
- R1: value 10k -> 270k
Connections:
- net GND: now also U2.13 (PS/SYNC)
- net at C5.1, U2.1 (VINA), U2.12 (EN): no longer U2.13 (PS/SYNC)
Changed lines of the file:
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@@
 	)
 	(junction
-		(at 152.4 43.18)
-		(diameter 0)
-		(color 0 0 0 0)
-	)
-	(junction
 		(at 129.54 170.18)
 		(diameter 0)
@@
 	)
 	(junction
+		(at 152.4 52.07)
+		(diameter 0)
+		(color 0 0 0 0)
+	)
+	(junction
 		(at 44.45 29.21)
 		(diameter 0)
@@
 	(wire
 		(pts
+			(xy 156.21 43.18) (xy 156.21 52.07)
+		)
+		(stroke
+			(width 0)
+			(type default)
+		)
+	)
+	(wire
+		(pts
 			(xy 270.51 146.05) (xy 260.35 146.05)
 		)
@@
 	(wire
 		(pts
-			(xy 152.4 50.8) (xy 152.4 49.53)
+			(xy 152.4 50.8) (xy 152.4 52.07)
 		)
 		(stroke
@@
 	(wire
 		(pts
+			(xy 156.21 52.07) (xy 152.4 52.07)
+		)
+		(stroke
+			(width 0)
+			(type default)
+		)
+	)
+	(wire
+		(pts
 			(xy 242.57 64.77) (xy 247.65 64.77)
 		)
@@
 	(wire
 		(pts
-			(xy 152.4 43.18) (xy 156.21 43.18)
-		)
-		(stroke
-			(width 0)
-			(type default)
-		)
-	)
-	(wire
-		(pts
 			(xy 82.55 39.37) (xy 59.69 39.37)
 		)
@@
 	(wire
 		(pts
+			(xy 152.4 52.07) (xy 152.4 53.34)
+		)
+		(stroke
+			(width 0)
+			(type default)
+		)
+	)
+	(wire
+		(pts
 			(xy 81.28 58.42) (xy 104.14 58.42)
 		)
@@
 			)
 		)
-		(property "Value" "10k"
+		(property "Value" "270k"
 			(at 207.01 148.59 0)
 			(effects
@@
 	(symbol
 		(lib_id "power:GND")
-		(at 152.4 49.53 0)
+		(at 152.4 53.34 0)
 		(unit 1)
 		(exclude_from_sim no)
@@
 		(dnp no)
 		(property "Reference" "#PWR05"
-			(at 152.4 55.88 0)
+			(at 152.4 59.69 0)
 			(effects
 				(font
@@
 		)
 		(property "Value" "GND"
-			(at 152.4 55.88 0)
+			(at 152.4 59.69 0)
 			(effects
 				(font
@@
 		)
 		(property "Footprint" ""
-			(at 152.4 49.53 0)
+			(at 152.4 53.34 0)
 			(effects
 				(font
@@
 		)
 		(property "Datasheet" ""
-			(at 152.4 49.53 0)
+			(at 152.4 53.34 0)
 			(effects
 				(font
@@
 		)
 		(property "Description" ""
-			(at 152.4 49.53 0)
+			(at 152.4 53.34 0)
 			(effects
 				(font

Commit message: Minor KiCad files update for all devices
Parts:
- C3: value 1nF -> 68nF
- R1: value 270k -> 200k
- R7: value 68k -> 75k
Other:
- title: HueMix-Link Motion Sensor -> HueMix-Link Magnetic Sensor
Changed lines of the file:
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@@
 	(paper "A4")
 	(title_block
-		(title "HueMix-Link Motion Sensor")
-		(date "2026-02-18")
+		(title "HueMix-Link Magnetic Sensor")
+		(date "2026-04-03")
 		(rev "1.0")
 	)
@@
 			)
 		)
-		(property "Value" "270k"
-			(at 207.01 148.59 0)
+		(property "Value" "200k"
+			(at 208.28 148.59 0)
 			(effects
 				(font
@@
 			)
 		)
-		(property "Value" "1nF"
+		(property "Value" "68nF"
 			(at 25.4 41.9099 0)
 			(effects
@@
 			)
 		)
-		(property "Value" "68k"
+		(property "Value" "75k"
 			(at 262.89 140.9699 0)
 			(effects

Commit message: Fix magnetic sensor pcb
Parts:
- U2: DESCRIPTION High Efficiency Single Inductor Buck-Boost Converter with 4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 -> (none)
